Commit message: urdf and mapping.launch updated

File: TKProject4/my_robot/urdf/my_robot.xacro (robot description, xacro)
@@ -71,4 +71,9 @@
     <axis xyz="0 1 0" rpy="0 0 0"/>
   </joint>
+  <joint name="camera_optical_joint" type="fixed">
+    <origin xyz="0 0 0" rpy="-1.5707 0 -1.5707"/>
+    <parent link="camera"/>
+    <child link="camera_link_optical"/>
+  </joint>
   <joint name="hokuyo_joint" type="fixed">
     <origin xyz="0.3 0 0.045" rpy="0 0 0"/>
@@ -332,4 +337,6 @@
     </visual>
   </link>
+  <link name="camera_link_optical">
+  </link>
   <link name='hokuyo'>
     <pose>0 0 0 0 0 0</pose>

Commit message: localization.launch and teleop.launch added, sim ss added

File: TKProject4/my_robot/urdf/my_robot.xacro (robot description, xacro)
@@ -71,14 +71,14 @@
     <axis xyz="0 1 0" rpy="0 0 0"/>
   </joint>
+  <joint name="hokuyo_joint" type="fixed">
+    <origin xyz="0.3 0 0.045" rpy="0 0 0"/>
+    <child link="hokuyo"/>
+    <parent link="body_part_roof"/>
+    <axis xyz="0 1 0" rpy="0 0 0"/>
+  </joint>
   <joint name="camera_optical_joint" type="fixed">
     <origin xyz="0 0 0" rpy="-1.5707 0 -1.5707"/>
     <parent link="camera"/>
     <child link="camera_link_optical"/>
-  </joint>
-  <joint name="hokuyo_joint" type="fixed">
-    <origin xyz="0.3 0 0.045" rpy="0 0 0"/>
-    <child link="hokuyo"/>
-    <parent link="body_part_roof"/>
-    <axis xyz="0 1 0" rpy="0 0 0"/>
   </joint>
   <!--Links-->
@@ -312,5 +312,4 @@
     </visual>
   </link>
-  <!--Camera-->
   <link name='camera'>
     <pose>0 0 0 0 0 0</pose>
